Commit message: DRC-2046: very critical bugfix in collision avoidance. Urdf Updated. wont fixBamboo

File: DarpaRoboticsChallenge/resources/models/atlas_v4_robotiq.wb.urdf (robot description, URDF)
Before this commit: robot drc_skeleton, 31 links, 30 joints
Links:
- link l_larm: geometry visual mesh filename=package://atlas_description/meshes_v3/l_larm.dae scale=1 1 1; visual sphere radius=0.09
- link l_uleg: geometry visual mesh filename=package://atlas_description/meshes_v3/l_uleg.dae scale=1 1 1; visual sphere radius=0.12
- link pelvis: geometry visual mesh filename=package://atlas_description/meshes_v3/pelvis.dae scale=1 1 1; visual sphere radius=0.20
- link r_larm: geometry visual mesh filename=package://atlas_description/meshes_v3/r_larm.dae scale=1 1 1; visual sphere radius=0.09
- link r_uleg: geometry visual mesh filename=package://atlas_description/meshes_v3/r_uleg.dae scale=1 1 1; visual sphere radius=0.12
- link utorso: geometry visual mesh filename=package://atlas_description/meshes_v3/utorso.dae scale=1 1 1; visual mesh filename=package://atlas_description/meshes_v3/utorso_pack.dae scale=1 1 1

Commit message: DRC-2046: minor fixes and urdf update. wont fixBamboo

File: DarpaRoboticsChallenge/resources/models/atlas_v4_robotiq.wb.urdf (robot description, URDF)
Before this commit: robot drc_skeleton, 31 links, 30 joints
Links:
- link utorso: geometry visual mesh filename=package://atlas_description/meshes_v3/utorso.dae scale=1 1 1; visual mesh filename=package://atlas_description/meshes_v3/utorso_pack.dae scale=1 1 1

Commit message: NONE: BOOOOOM! Big dangerous and no-one-asked-to-do-that commit. will probably brake Bamboo and most definitely won't fixBamboo,
Methods in JMEGeometryUtils have been changed, affecting many callers.
The behavior of SDFFullRobotModel.getEndEffectorFrame is different and ModifiableCylinderGrabber changed accordingly.

File: DarpaRoboticsChallenge/resources/models/atlas_v4_robotiq.wb.urdf (robot description, URDF)
Before this commit: robot drc_skeleton, 31 links, 30 joints
Joints:
- joint l_ee_fixed_joint: origin xyz=0  0.26  0 rpy=-1.5708 0 1.5708 -> xyz=0  0.26  0 rpy=0 0 0
- joint r_ee_fixed_joint: origin xyz=-0.0 -0.26  -0.00 rpy=1.5708 0 -1.5708 -> xyz=0 -0.26  0 rpy=0 0 0

Commit message: NONE: returning to old coordinates for the hand... hopefully. might fixBamboo

File: DarpaRoboticsChallenge/resources/models/atlas_v4_robotiq.wb.urdf (robot description, URDF)
Before this commit: robot drc_skeleton, 31 links, 30 joints
Joints:
- joint l_ee_fixed_joint: origin xyz=0  0.26  0 rpy=0 0 0 -> xyz=0  0.26  0 rpy=-1.5708 0 1.5708
- joint r_ee_fixed_joint: origin xyz=0 -0.26  0 rpy=0 0 0 -> xyz=0 -0.26  0 rpy=1.5708 0 -1.5708

Commit message: NONE: important fix in the URDF. r_leg_hipz was wrongly placed. might fixBamboo

File: DarpaRoboticsChallenge/resources/models/atlas_v4_robotiq.wb.urdf (robot description, URDF)
Before this commit: robot drc_skeleton, 31 links, 30 joints
Joints:
- joint back_bkz: origin xyz=-0.0125 0 0 rpy=0 -0 0 -> xyz=-0.0125 0.089 0 rpy=0 -0 0
- joint l_leg_hpz: origin xyz=0 0.089 0 rpy=0 -0 0 -> xyz=0 0.178 0 rpy=0 -0 0
- joint r_leg_hpz: origin xyz=0 0.089 0 rpy=0 -0 0 -> xyz=0 0 0 rpy=0 -0 0
