Commit message: DRC-2505: changing plugin back to force control and handless for now. incorporating estimator dt in timing. won't fixBamboo

File: Atlas/ihmc_gazebo_catkin_ws/src/ihmc_gazebo/urdf/atlas_v4_no_wry2_simple_shapes.urdf (robot description, URDF)
Before this commit: robot drc_skeleton, 32 links, 32 joints
Links:
- link l_lglut: geometry collision box size=0.125 0.05 0.08; collision cylinder length=0.060306 radius=0.02009687
- link l_uglut: geometry collision box size=0.05 0.1 0.1; collision cylinder length=0.080842 radius=0.019841
- link r_lglut: geometry collision box size=0.125 0.05 0.08; collision cylinder length=0.060306 radius=0.02009687
- link r_uglut: geometry collision box size=0.05 0.1 0.1; collision cylinder length=0.080842 radius=0.019841
- link utorso: geometry collision box size=0.13 0.50 0.10; collision box size=0.2 0.18 0.10

File: Atlas/ihmc_gazebo_catkin_ws/src/ihmc_gazebo/urdf/atlas_v5_simple_shapes.urdf (robot description, URDF)
Before this commit: robot drc_skeleton, 34 links, 34 joints
Links:
- link l_lglut: geometry collision box size=0.0975 0.069 0.103; collision cylinder length=0.060306 radius=0.02009687
- link l_uglut: geometry collision cylinder length=0.078396 radius=0.019096; collision cylinder length=0.080842 radius=0.019841
- link r_lglut: geometry collision box size=0.0975 0.069 0.103; collision cylinder length=0.060306 radius=0.02009687
- link r_uglut: geometry collision cylinder length=0.078396 radius=0.019096; collision cylinder length=0.080842 radius=0.019841
- link utorso: geometry collision box size=0.2 0.25 0.01; collision box size=0.456306 0.341719 0.12

File: Atlas/ihmc_gazebo_catkin_ws/src/ihmc_gazebo/urdf/ihmc_atlas_v5.urdf.xacro (robot description, xacro)
@@ -1,11 +1,4 @@
 <robot xmlns:xacro="http://www.ros.org/wiki/xacro" name="atlas" >
-    <xacro:include filename="$(find ihmc_gazebo)/urdf/atlas_v5.urdf" />
-    <xacro:include filename="$(find ihmc_gazebo)/urdf/robotiq_hand.urdf.xacro" />
-    <xacro:robotiq_hand prefix="l_" parent="l_hand" reflect="-1">
-    	<origin rpy="3.14159 3.14159 3.14159" xyz="-0.00125 0.17 0.01"/>
-  	</xacro:robotiq_hand>
-  	<xacro:robotiq_hand prefix="r_" parent="r_hand" reflect="1">
-    	<origin rpy="3.14159 0 0" xyz="-0.00125 -0.17 0.01"/>
-  	</xacro:robotiq_hand>
+    <xacro:include filename="$(find ihmc_gazebo)/urdf/atlas_v5_simple_shapes.urdf" />
     <xacro:include filename="$(find ihmc_gazebo)/urdf/atlas_v5.gazebo" />
     <xacro:include filename="$(find atlas_description)/urdf/atlas_v5.transmission" />
