Commit message: ROSI-72: imported new Val models; chest orientation is behaving properly for now; won't fixbamboo

File: resources/models/val_description/robots/valkyrie_A/xacro/arm/arm.xacro (robot description, xacro)
@@ -175,5 +175,5 @@
   </xacro:macro>
   <!-- Actuators -->
-  <xacro:macro name="v1_upper_arm_actuators" params="name1 type1 name2 type2 name3 type3 name4 type4">
+  <xacro:macro name="upper_arm_actuators" params="name1 type1 name2 type2 name3 type3 name4 type4">
     <actuator name="${name1}" type="${type1}"/>
     <actuator name="${name2}" type="${type2}"/>
@@ -181,12 +181,12 @@
     <actuator name="${name4}" type="${type4}"/>
   </xacro:macro>
-  <xacro:macro name="v1_lower_arm_actuators" params="name1 type1 name2 type2 name3 type3">
+  <xacro:macro name="lower_arm_actuators" params="name1 type1 name2 type2 name3 type3">
     <actuator name="${name1}" type="${type1}"/>
     <actuator name="${name2}" type="${type2}"/>
     <actuator name="${name3}" type="${type3}"/>
   </xacro:macro>
-  <xacro:macro name="v1_arm_actuators" params="name1 type1 name2 type2 name3 type3 name4 type4 name5 type5 name6 type6 name7 type7">
-    <xacro:v1_upper_arm_actuators name1="${name1}" type1="${type1}" name2="${name2}" type2="${type2}" name3="${name3}" type3="${type3}" name4="${name4}" type4="${type4}"/>
-    <xacro:v1_lower_arm_actuators name1="${name5}" type1="${type5}" name2="${name6}" type2="${type6}" name3="${name7}" type3="${type7}" />
+  <xacro:macro name="arm_actuators" params="name1 type1 name2 type2 name3 type3 name4 type4 name5 type5 name6 type6 name7 type7">
+    <xacro:upper_arm_actuators name1="${name1}" type1="${type1}" name2="${name2}" type2="${type2}" name3="${name3}" type3="${type3}" name4="${name4}" type4="${type4}"/>
+    <xacro:lower_arm_actuators name1="${name5}" type1="${type5}" name2="${name6}" type2="${type6}" name3="${name7}" type3="${type7}" />
   </xacro:macro>
 </robot>

File: resources/models/val_description/robots/valkyrie_A/xacro/head/head.xacro (robot description, xacro)
@@ -6,5 +6,4 @@
   <xacro:include filename="$(find val_description)/robots/valkyrie_A/xacro/head/frame_parameters.xacro"/>
   <xacro:include filename="$(find val_description)/robots/valkyrie_A/xacro/head/mass_parameters.xacro"/>
-  <xacro:include filename="$(find val_description)/robots/common/sensors/multisense_sl.xacro"/>
   <xacro:property name="NJ3_Link_Radius" value="0.139"/>
   <xacro:macro name="include_head" params="lower_neck_pitch_root_link">
@@ -52,18 +51,9 @@
       <controller_gains Kp="20000" Kd="0"/>
     </xacro:revolute_joint_ex>
-  </xacro:macro>
-  <xacro:macro name="v1_head_sensors">
-    <xacro:multisense_sl parentLink="${UpperNeckPitchLinkName}"
-                  joint_axis="1 0 0"
-                  joint_origin_xyz="${HokuyoFrameOrigin_X} ${HokuyoFrameOrigin_Y} ${HokuyoFrameOrigin_Z}"
-                  joint_origin_rpy="${HokuyoFrameOrientation_Roll} ${HokuyoFrameOrientation_Pitch} ${HokuyoFrameOrientation_Yaw}"
-                  com_origin_xyz="${HokuyoLinkComPosition}"
-                  com_origin_rpy="0 0 0"
-                  mass="${HokuyoLinkMass}"
-                  visual_mesh="${mesh_root}/head/multisense_hokuyo.dae"
-                  material="White"
-                  collision_mesh="${mesh_root}/head/multisense_hokuyo.dae" />
-  </xacro:macro>
-  <xacro:macro name="v1_head_actuators" params="name1 type1 name2 type2 name3 type3">
+    </xacro:macro>
+    <xacro:macro name="include_multisense">
+      <xacro:fixed_joint jointName="multisense_head_root" parent="${UpperNeckPitchLinkName}" child="head" origin_xyz="0.183585961 0.0 0.075353826" origin_rpy="-3.14159 0.130899694 0.0" />
+    </xacro:macro>
+  <xacro:macro name="neck_actuators" params="name1 type1 name2 type2 name3 type3">
     <actuator name="${name1}" type="${type1}"/>
     <actuator name="${name2}" type="${type2}"/>

File: resources/models/val_description/robots/valkyrie_A/xacro/head/link_names.xacro (robot description, xacro)
@@ -4,4 +4,4 @@
   <xacro:property name="LowerNeckPitchLinkName" value="LowerNeckPitchLink" />
   <xacro:property name="NeckYawLinkName" value="NeckYawLink" />
-  <xacro:property name="UpperNeckPitchLinkName" value="Head" />
+  <xacro:property name="UpperNeckPitchLinkName" value="UpperNeckPitchLinkName" />
 </robot>

File: resources/models/val_description/robots/valkyrie_A/xacro/index_finger/index_finger.xacro (robot description, xacro)
@@ -44,5 +44,10 @@
                           origin_rpy="${IndexFingerPitch1FrameOrientation_Roll} ${IndexFingerPitch1FrameOrientation_Pitch} ${IndexFingerPitch1FrameOrientation_Yaw}"
                           axis="${IndexFingerPitch1RotationAxis}">
-        <limit effort="${IndexFingerPitch1TorqueLimit}" lower="${IndexFingerPitch1PositionLimit_Lower}" upper="${IndexFingerPitch1PositionLimit_Upper}" velocity="${IndexFingerPitch1VelocityLimit}"/>
+        <xacro:if value="${(reflect+1)/2}">
+          <limit effort="${IndexFingerPitch1TorqueLimit}" lower="${-reflect * IndexFingerPitch1PositionLimit_Upper}" upper="${-reflect * IndexFingerPitch1PositionLimit_Lower}" velocity="${IndexFingerPitch1VelocityLimit}"/>
+        </xacro:if>
+        <xacro:if value="${(-reflect+1)/2}">
+          <limit effort="${IndexFingerPitch1TorqueLimit}" lower="${IndexFingerPitch1PositionLimit_Lower}" upper="${IndexFingerPitch1PositionLimit_Upper}" velocity="${IndexFingerPitch1VelocityLimit}"/>
+        </xacro:if>
     </xacro:revolute_joint>
     <xacro:revolute_joint jointName="${IndexFingerPitch2JointName}"
@@ -51,5 +56,10 @@
                           origin_rpy="${IndexFingerPitch2FrameOrientation_Roll} ${IndexFingerPitch2FrameOrientation_Pitch} ${IndexFingerPitch2FrameOrientation_Yaw}"
                           axis="${IndexFingerPitch2RotationAxis}">
-        <limit effort="${IndexFingerPitch2TorqueLimit}" lower="${IndexFingerPitch2PositionLimit_Lower}" upper="${IndexFingerPitch2PositionLimit_Upper}" velocity="${IndexFingerPitch2VelocityLimit}"/>
+        <xacro:if value="${(reflect+1)/2}">
+          <limit effort="${IndexFingerPitch2TorqueLimit}" lower="${-reflect * IndexFingerPitch2PositionLimit_Upper}" upper="${-reflect * IndexFingerPitch2PositionLimit_Lower}" velocity="${IndexFingerPitch2VelocityLimit}"/>
+        </xacro:if>
+        <xacro:if value="${(-reflect+1)/2}">
+          <limit effort="${IndexFingerPitch2TorqueLimit}" lower="${IndexFingerPitch2PositionLimit_Lower}" upper="${IndexFingerPitch2PositionLimit_Upper}" velocity="${IndexFingerPitch2VelocityLimit}"/>
+        </xacro:if>
     </xacro:revolute_joint>
     <xacro:revolute_joint jointName="${IndexFingerPitch3JointName}"
@@ -58,5 +68,10 @@
                           origin_rpy="${IndexFingerPitch3FrameOrientation_Roll} ${IndexFingerPitch3FrameOrientation_Pitch} ${IndexFingerPitch3FrameOrientation_Yaw}"
                           axis="${IndexFingerPitch3RotationAxis}">
-        <limit effort="${IndexFingerPitch3TorqueLimit}" lower="${IndexFingerPitch3PositionLimit_Lower}" upper="${IndexFingerPitch3PositionLimit_Upper}" velocity="${IndexFingerPitch3VelocityLimit}"/>
+        <xacro:if value="${(reflect+1)/2}">
+          <limit effort="${IndexFingerPitch3TorqueLimit}" lower="${-reflect * IndexFingerPitch3PositionLimit_Upper}" upper="${-reflect * IndexFingerPitch3PositionLimit_Lower}" velocity="${IndexFingerPitch3VelocityLimit}"/>
+        </xacro:if>
+        <xacro:if value="${(-reflect+1)/2}">
+          <limit effort="${IndexFingerPitch3TorqueLimit}" lower="${IndexFingerPitch3PositionLimit_Lower}" upper="${IndexFingerPitch3PositionLimit_Upper}" velocity="${IndexFingerPitch3VelocityLimit}"/>
+        </xacro:if>
     </xacro:revolute_joint>
   </xacro:macro>

File: resources/models/val_description/robots/valkyrie_A/xacro/index_finger/joint_limits.xacro (robot description, xacro)
@@ -5,12 +5,12 @@
   <xacro:property name="IndexFingerPitch3TorqueLimit" value="10" />
   <xacro:property name="IndexFingerPitch4TorqueLimit" value="10" />
-  <xacro:property name="IndexFingerPitch1PositionLimit_Lower" value="-0.087" />
-  <xacro:property name="IndexFingerPitch2PositionLimit_Lower" value="-1.658" />
-  <xacro:property name="IndexFingerPitch3PositionLimit_Lower" value="-1.920" />
-  <xacro:property name="IndexFingerPitch4PositionLimit_Lower" value="-1.57" />
-  <xacro:property name="IndexFingerPitch1PositionLimit_Upper" value="0.087" />
-  <xacro:property name="IndexFingerPitch2PositionLimit_Upper" value="0.175" />
-  <xacro:property name="IndexFingerPitch3PositionLimit_Upper" value="0" />
-  <xacro:property name="IndexFingerPitch4PositionLimit_Upper" value="0.175" />
+  <xacro:property name="IndexFingerPitch1PositionLimit_Lower" value="0.0" />
+  <xacro:property name="IndexFingerPitch2PositionLimit_Lower" value="0.0" />
+  <xacro:property name="IndexFingerPitch3PositionLimit_Lower" value="0.0" />
+  <xacro:property name="IndexFingerPitch4PositionLimit_Lower" value="0.0" />
+  <xacro:property name="IndexFingerPitch1PositionLimit_Upper" value="1.57" />
+  <xacro:property name="IndexFingerPitch2PositionLimit_Upper" value="1.658" />
+  <xacro:property name="IndexFingerPitch3PositionLimit_Upper" value="1.920" />
+  <xacro:property name="IndexFingerPitch4PositionLimit_Upper" value="1.57" />
   <xacro:property name="IndexFingerPitch1VelocityLimit" value="1" />
   <xacro:property name="IndexFingerPitch2VelocityLimit" value="1" />

File: resources/models/val_description/robots/valkyrie_A/xacro/leg/leg.xacro (robot description, xacro)
@@ -14,7 +14,4 @@
   <xacro:property name="LJ1_Link_Origin_Y" value="0.0013"/>
   <xacro:property name="LJ1_Link_Origin_Z" value="0.03867"/>
-  <!-- <xacro:property name="LJ1_Link_Origin_X" value="1.3078570e-03"/>
-  <xacro:property name="LJ1_Link_Origin_Y" value="2.1764163e-02"/>
-  <xacro:property name="LJ1_Link_Origin_Z" value="3.8670367e-02"/> -->
   <xacro:property name="LJ2_Link_Width" value="0.123"/>
   <xacro:property name="LJ2_Link_Height" value="0.131"/>
@@ -74,13 +71,4 @@
                     material="White"
                     collision_mesh="${mesh_root}/legs/foot_${prefix}.dae" />
-    <gazebo reference="${AnkleRollLinkName}">
-      <kp>100000.0</kp>
-      <kd>1000.0</kd>
-      <mu1>1.5</mu1>
-      <mu2>1.5</mu2>
-      <fdir1>0 0 1</fdir1>
-      <maxVel>1.0</maxVel>
-      <minDepth>0.00</minDepth>
-    </gazebo>
   </xacro:macro>
   <xacro:macro name="make_leg_joints" params="prefix reflect leg_root_link">
@@ -169,5 +157,5 @@
                         origin_rpy="3.14 0.0 -1.047"/>
   </xacro:macro>
-  <xacro:macro name="v1_leg_actuators" params="name1 type1 name2 type2 name3 type3 name4 type4 name5 type5 name6 type6">
+  <xacro:macro name="leg_actuators" params="name1 type1 name2 type2 name3 type3 name4 type4 name5 type5 name6 type6">
     <actuator name="${name1}" type="${type1}"/>
     <actuator name="${name2}" type="${type2}"/>
@@ -177,13 +165,3 @@
     <actuator name="${name6}" type="${type6}"/>
   </xacro:macro>
-  <xacro:macro name="v1_leg_actuators_no_ankle" params="name1 type1 name2 type2 name3 type3 name4 type4">
-    <actuator name="${name1}" type="${type1}"/>
-    <actuator name="${name2}" type="${type2}"/>
-    <actuator name="${name3}" type="${type3}"/>
-    <actuator name="${name4}" type="${type4}"/>
-  </xacro:macro>
-  <xacro:macro name="v1_ankle_actuators" params="name5 type5 name6 type6">
-    <actuator name="${name5}" type="${type5}"/>
-    <actuator name="${name6}" type="${type6}"/>
-  </xacro:macro>
 </robot>

File: resources/models/val_description/robots/valkyrie_A/xacro/middle_finger/joint_limits.xacro (robot description, xacro)
@@ -4,10 +4,10 @@
   <xacro:property name="MiddleFingerPitch2TorqueLimit" value="10" />
   <xacro:property name="MiddleFingerPitch3TorqueLimit" value="10" />
-  <xacro:property name="MiddleFingerPitch1PositionLimit_Lower" value="-1.658" />
-  <xacro:property name="MiddleFingerPitch2PositionLimit_Lower" value="-1.920" />
-  <xacro:property name="MiddleFingerPitch3PositionLimit_Lower" value="-1.57" />
-  <xacro:property name="MiddleFingerPitch1PositionLimit_Upper" value="0.175" />
-  <xacro:property name="MiddleFingerPitch2PositionLimit_Upper" value="0" />
-  <xacro:property name="MiddleFingerPitch3PositionLimit_Upper" value="0.175" />
+  <xacro:property name="MiddleFingerPitch1PositionLimit_Upper" value="1.658" />
+  <xacro:property name="MiddleFingerPitch2PositionLimit_Upper" value="1.920" />
+  <xacro:property name="MiddleFingerPitch3PositionLimit_Upper" value="1.57" />
+  <xacro:property name="MiddleFingerPitch1PositionLimit_Lower" value="0.0" />
+  <xacro:property name="MiddleFingerPitch2PositionLimit_Lower" value="0.0" />
+  <xacro:property name="MiddleFingerPitch3PositionLimit_Lower" value="0.0" />
   <xacro:property name="MiddleFingerPitch1VelocityLimit" value="1" />
   <xacro:property name="MiddleFingerPitch2VelocityLimit" value="1" />

File: resources/models/val_description/robots/valkyrie_A/xacro/middle_finger/middle_finger.xacro (robot description, xacro)
@@ -44,5 +44,10 @@
                           origin_rpy="${MiddleFingerPitch1FrameOrientation_Roll} ${MiddleFingerPitch1FrameOrientation_Pitch} ${MiddleFingerPitch1FrameOrientation_Yaw}"
                           axis="${MiddleFingerPitch1RotationAxis}">
-        <limit effort="${MiddleFingerPitch1TorqueLimit}" lower="${MiddleFingerPitch1PositionLimit_Lower}" upper="${MiddleFingerPitch1PositionLimit_Upper}" velocity="${MiddleFingerPitch1VelocityLimit}"/>
+        <xacro:if value="${(reflect+1)/2}">
+          <limit effort="${MiddleFingerPitch1TorqueLimit}" lower="${-reflect * MiddleFingerPitch1PositionLimit_Upper}" upper="${-reflect * MiddleFingerPitch1PositionLimit_Lower}" velocity="${MiddleFingerPitch1VelocityLimit}"/>
+        </xacro:if>
+        <xacro:if value="${(-reflect+1)/2}">
+          <limit effort="${MiddleFingerPitch1TorqueLimit}" lower="${MiddleFingerPitch1PositionLimit_Lower}" upper="${MiddleFingerPitch1PositionLimit_Upper}" velocity="${MiddleFingerPitch1VelocityLimit}"/>
+        </xacro:if>
     </xacro:revolute_joint>
     <xacro:revolute_joint jointName="${MiddleFingerPitch2JointName}"
@@ -51,5 +56,10 @@
                           origin_rpy="${MiddleFingerPitch2FrameOrientation_Roll} ${MiddleFingerPitch2FrameOrientation_Pitch} ${MiddleFingerPitch2FrameOrientation_Yaw}"
                           axis="${MiddleFingerPitch2RotationAxis}">
-        <limit effort="${MiddleFingerPitch2TorqueLimit}" lower="${MiddleFingerPitch2PositionLimit_Lower}" upper="${MiddleFingerPitch2PositionLimit_Upper}" velocity="${MiddleFingerPitch2VelocityLimit}"/>
+        <xacro:if value="${(reflect+1)/2}">
+          <limit effort="${MiddleFingerPitch2TorqueLimit}" lower="${-reflect * MiddleFingerPitch2PositionLimit_Upper}" upper="${-reflect * MiddleFingerPitch2PositionLimit_Lower}" velocity="${MiddleFingerPitch2VelocityLimit}"/>
+        </xacro:if>
+        <xacro:if value="${(-reflect+1)/2}">
+          <limit effort="${MiddleFingerPitch2TorqueLimit}" lower="${MiddleFingerPitch2PositionLimit_Lower}" upper="${MiddleFingerPitch2PositionLimit_Upper}" velocity="${MiddleFingerPitch2VelocityLimit}"/>
+        </xacro:if>
     </xacro:revolute_joint>
     <xacro:revolute_joint jointName="${MiddleFingerPitch3JointName}"
@@ -58,5 +68,10 @@
                           origin_rpy="${MiddleFingerPitch3FrameOrientation_Roll} ${MiddleFingerPitch3FrameOrientation_Pitch} ${MiddleFingerPitch3FrameOrientation_Yaw}"
                           axis="${MiddleFingerPitch3RotationAxis}">
-        <limit effort="${MiddleFingerPitch3TorqueLimit}" lower="${MiddleFingerPitch3PositionLimit_Lower}" upper="${MiddleFingerPitch3PositionLimit_Upper}" velocity="${MiddleFingerPitch3VelocityLimit}"/>
+        <xacro:if value="${(reflect+1)/2}">
+          <limit effort="${MiddleFingerPitch3TorqueLimit}" lower="${-reflect * MiddleFingerPitch3PositionLimit_Upper}" upper="${-reflect * MiddleFingerPitch3PositionLimit_Lower}" velocity="${MiddleFingerPitch3VelocityLimit}"/>
+        </xacro:if>
+        <xacro:if value="${(-reflect+1)/2}">
+          <limit effort="${MiddleFingerPitch3TorqueLimit}" lower="${MiddleFingerPitch3PositionLimit_Lower}" upper="${MiddleFingerPitch3PositionLimit_Upper}" velocity="${MiddleFingerPitch3VelocityLimit}"/>
+        </xacro:if>
     </xacro:revolute_joint>
   </xacro:macro>

File: resources/models/val_description/robots/valkyrie_A/xacro/pinky_finger/joint_limits.xacro (robot description, xacro)
@@ -1,19 +1,15 @@
 <?xml version="1.0" ?>
 <robot xmlns:xacro="http://www.ros.org/wiki/xacro" name="v1/pinky_finger/joint_limits">
-  <xacro:property name="PinkyPitch1TorqueLimit" value="10" />
-  <xacro:property name="PinkyPitch2TorqueLimit" value="10" />
-  <xacro:property name="PinkyPitch3TorqueLimit" value="10" />
-  <xacro:property name="PinkyPitch4TorqueLimit" value="10" />
-  <xacro:property name="PinkyPitch1PositionLimit_Lower" value="-0.262" />
-  <xacro:property name="PinkyPitch2PositionLimit_Lower" value="-1.658" />
-  <xacro:property name="PinkyPitch3PositionLimit_Lower" value="-1.920" />
-  <xacro:property name="PinkyPitch4PositionLimit_Lower" value="-1.57" />
-  <xacro:property name="PinkyPitch1PositionLimit_Upper" value="0.0" />
-  <xacro:property name="PinkyPitch2PositionLimit_Upper" value="0.175" />
-  <xacro:property name="PinkyPitch3PositionLimit_Upper" value="0" />
-  <xacro:property name="PinkyPitch4PositionLimit_Upper" value="0.175" />
-  <xacro:property name="PinkyPitch1VelocityLimit" value="1" />
-  <xacro:property name="PinkyPitch2VelocityLimit" value="1" />
-  <xacro:property name="PinkyPitch3VelocityLimit" value="1" />
-  <xacro:property name="PinkyPitch4VelocityLimit" value="1" />
+  <xacro:property name="PinkyFingerPitch1TorqueLimit" value="10" />
+  <xacro:property name="PinkyFingerPitch2TorqueLimit" value="10" />
+  <xacro:property name="PinkyFingerPitch3TorqueLimit" value="10" />
+  <xacro:property name="PinkyFingerPitch1PositionLimit_Lower" value="0.0" />
+  <xacro:property name="PinkyFingerPitch2PositionLimit_Lower" value="0.0" />
+  <xacro:property name="PinkyFingerPitch3PositionLimit_Lower" value="0.0" />
+  <xacro:property name="PinkyFingerPitch1PositionLimit_Upper" value="1.57" />
+  <xacro:property name="PinkyFingerPitch2PositionLimit_Upper" value="1.658" />
+  <xacro:property name="PinkyFingerPitch3PositionLimit_Upper" value="1.920" />
+  <xacro:property name="PinkyFingerPitch1VelocityLimit" value="1" />
+  <xacro:property name="PinkyFingerPitch2VelocityLimit" value="1" />
+  <xacro:property name="PinkyFingerPitch3VelocityLimit" value="1" />
 </robot>

File: resources/models/val_description/robots/valkyrie_A/xacro/pinky_finger/pinky_finger.xacro (robot description, xacro)
@@ -44,5 +44,10 @@
                           origin_rpy="${PinkyPitch1FrameOrientation_Roll} ${PinkyPitch1FrameOrientation_Pitch} ${PinkyPitch1FrameOrientation_Yaw}"
                           axis="${PinkyFingerPitch1RotationAxis}">
-        <limit effort="${PinkyPitch1TorqueLimit}" lower="${PinkyPitch1PositionLimit_Lower}" upper="${PinkyPitch1PositionLimit_Upper}" velocity="${PinkyPitch1VelocityLimit}"/>
+        <xacro:if value="${(reflect+1)/2}">
+          <limit effort="${PinkyFingerPitch1TorqueLimit}" lower="${-reflect * PinkyFingerPitch1PositionLimit_Upper}" upper="${-reflect * PinkyFingerPitch1PositionLimit_Lower}" velocity="${PinkyFingerPitch1VelocityLimit}"/>
+        </xacro:if>
+        <xacro:if value="${(-reflect+1)/2}">
+          <limit effort="${PinkyFingerPitch1TorqueLimit}" lower="${PinkyFingerPitch1PositionLimit_Lower}" upper="${PinkyFingerPitch1PositionLimit_Upper}" velocity="${PinkyFingerPitch1VelocityLimit}"/>
+        </xacro:if>
     </xacro:revolute_joint>
     <xacro:revolute_joint jointName="${PinkyPitch2JointName}"
@@ -51,5 +56,10 @@
                           origin_rpy="${PinkyPitch2FrameOrientation_Roll} ${PinkyPitch2FrameOrientation_Pitch} ${PinkyPitch2FrameOrientation_Yaw}"
                           axis="${PinkyFingerPitch2RotationAxis}">
-        <limit effort="${PinkyPitch2TorqueLimit}" lower="${PinkyPitch2PositionLimit_Lower}" upper="${PinkyPitch2PositionLimit_Upper}" velocity="${PinkyPitch2VelocityLimit}"/>
+        <xacro:if value="${(reflect+1)/2}">
+          <limit effort="${PinkyFingerPitch2TorqueLimit}" lower="${-reflect * PinkyFingerPitch2PositionLimit_Upper}" upper="${-reflect * PinkyFingerPitch2PositionLimit_Lower}" velocity="${PinkyFingerPitch2VelocityLimit}"/>
+        </xacro:if>
+        <xacro:if value="${(-reflect+1)/2}">
+          <limit effort="${PinkyFingerPitch2TorqueLimit}" lower="${PinkyFingerPitch2PositionLimit_Lower}" upper="${PinkyFingerPitch2PositionLimit_Upper}" velocity="${PinkyFingerPitch2VelocityLimit}"/>
+        </xacro:if>
     </xacro:revolute_joint>
     <xacro:revolute_joint jointName="${PinkyPitch3JointName}"
@@ -58,5 +68,10 @@
                           origin_rpy="${PinkyPitch3FrameOrientation_Roll} ${PinkyPitch3FrameOrientation_Pitch} ${PinkyPitch3FrameOrientation_Yaw}"
                           axis="${PinkyFingerPitch3RotationAxis}">
-        <limit effort="${PinkyPitch3TorqueLimit}" lower="${PinkyPitch3PositionLimit_Lower}" upper="${PinkyPitch3PositionLimit_Upper}" velocity="${PinkyPitch3VelocityLimit}"/>
+        <xacro:if value="${(reflect+1)/2}">
+          <limit effort="${PinkyFingerPitch3TorqueLimit}" lower="${-reflect * PinkyFingerPitch3PositionLimit_Upper}" upper="${-reflect * PinkyFingerPitch3PositionLimit_Lower}" velocity="${PinkyFingerPitch3VelocityLimit}"/>
+        </xacro:if>
+        <xacro:if value="${(-reflect+1)/2}">
+          <limit effort="${PinkyFingerPitch3TorqueLimit}" lower="${PinkyFingerPitch3PositionLimit_Lower}" upper="${PinkyFingerPitch3PositionLimit_Upper}" velocity="${PinkyFingerPitch3VelocityLimit}"/>
+        </xacro:if>
     </xacro:revolute_joint>
   </xacro:macro>
