Commit message: ROSI-72: imported new Val models; chest orientation is behaving properly for now; won't fixbamboo

File: resources/models/val_description/robots/valkyrie_A/xacro/thumb/joint_limits.xacro (robot description, xacro)
@@ -5,12 +5,12 @@
   <xacro:property name="ThumbPitch2TorqueLimit" value="10" />
   <xacro:property name="ThumbPitch3TorqueLimit" value="10" />
-  <xacro:property name="ThumbRollPositionLimit_Lower" value="-0.087" />
-  <xacro:property name="ThumbPitch1PositionLimit_Lower" value="-1.658" />
-  <xacro:property name="ThumbPitch2PositionLimit_Lower" value="-1.920" />
-  <xacro:property name="ThumbPitch3PositionLimit_Lower" value="-1.57" />
+  <xacro:property name="ThumbRollPositionLimit_Lower" value="0.0" />
+  <xacro:property name="ThumbPitch1PositionLimit_Lower" value="0.0" />
+  <xacro:property name="ThumbPitch2PositionLimit_Lower" value="0.0" />
+  <xacro:property name="ThumbPitch3PositionLimit_Lower" value="0.0" />
   <xacro:property name="ThumbRollPositionLimit_Upper" value="2.356" />
-  <xacro:property name="ThumbPitch1PositionLimit_Upper" value="0.175" />
-  <xacro:property name="ThumbPitch2PositionLimit_Upper" value="0.0" />
-  <xacro:property name="ThumbPitch3PositionLimit_Upper" value="0.175" />
+  <xacro:property name="ThumbPitch1PositionLimit_Upper" value="1.658" />
+  <xacro:property name="ThumbPitch2PositionLimit_Upper" value="1.920" />
+  <xacro:property name="ThumbPitch3PositionLimit_Upper" value="1.57" />
   <xacro:property name="ThumbRollVelocityLimit" value="1" />
   <xacro:property name="ThumbPitch1VelocityLimit" value="1" />

File: resources/models/val_description/robots/valkyrie_A/xacro/thumb/thumb.xacro (robot description, xacro)
@@ -61,5 +61,10 @@
                           origin_rpy="${ThumbPitch1FrameOrientation_Roll} ${ThumbPitch1FrameOrientation_Pitch} ${ThumbPitch1FrameOrientation_Yaw}"
                           axis="${ThumbPitch1RotationAxis}">
-        <limit effort="${ThumbPitch1TorqueLimit}" lower="${ThumbPitch1PositionLimit_Lower}" upper="${ThumbPitch1PositionLimit_Upper}" velocity="${ThumbPitch1VelocityLimit}"/>
+        <xacro:if value="${(reflect+1)/2}">
+          <limit effort="${ThumbPitch1TorqueLimit}" lower="${-reflect * ThumbPitch1PositionLimit_Upper}" upper="${-reflect * ThumbPitch1PositionLimit_Lower}" velocity="${ThumbPitch1VelocityLimit}"/>
+        </xacro:if>
+        <xacro:if value="${(-reflect+1)/2}">
+          <limit effort="${ThumbPitch1TorqueLimit}" lower="${ThumbPitch1PositionLimit_Lower}" upper="${ThumbPitch1PositionLimit_Upper}" velocity="${ThumbPitch1VelocityLimit}"/>
+        </xacro:if>
     </xacro:revolute_joint>
     <xacro:revolute_joint jointName="${ThumbPitch2JointName}"
@@ -68,5 +73,10 @@
                           origin_rpy="${ThumbPitch2FrameOrientation_Roll} ${ThumbPitch2FrameOrientation_Pitch} ${ThumbPitch2FrameOrientation_Yaw}"
                           axis="${ThumbPitch2RotationAxis}">
-        <limit effort="${ThumbPitch2TorqueLimit}" lower="${ThumbPitch2PositionLimit_Lower}" upper="${ThumbPitch2PositionLimit_Upper}" velocity="${ThumbPitch2VelocityLimit}"/>
+        <xacro:if value="${(reflect+1)/2}">
+          <limit effort="${ThumbPitch2TorqueLimit}" lower="${-reflect * ThumbPitch2PositionLimit_Upper}" upper="${-reflect * ThumbPitch2PositionLimit_Lower}" velocity="${ThumbPitch2VelocityLimit}"/>
+        </xacro:if>
+        <xacro:if value="${(-reflect+1)/2}">
+          <limit effort="${ThumbPitch2TorqueLimit}" lower="${ThumbPitch2PositionLimit_Lower}" upper="${ThumbPitch2PositionLimit_Upper}" velocity="${ThumbPitch2VelocityLimit}"/>
+        </xacro:if>
     </xacro:revolute_joint>
     <xacro:revolute_joint jointName="${ThumbPitch3JointName}"
@@ -75,5 +85,10 @@
                           origin_rpy="${ThumbPitch3FrameOrientation_Roll} ${ThumbPitch3FrameOrientation_Pitch} ${ThumbPitch3FrameOrientation_Yaw}"
                           axis="${ThumbPitch3RotationAxis}">
-        <limit effort="${ThumbPitch3TorqueLimit}" lower="${ThumbPitch3PositionLimit_Lower}" upper="${ThumbPitch3PositionLimit_Upper}" velocity="${ThumbPitch3VelocityLimit}"/>
+        <xacro:if value="${(reflect+1)/2}">
+          <limit effort="${ThumbPitch3TorqueLimit}" lower="${-reflect * ThumbPitch3PositionLimit_Upper}" upper="${-reflect * ThumbPitch3PositionLimit_Lower}" velocity="${ThumbPitch3VelocityLimit}"/>
+        </xacro:if>
+        <xacro:if value="${(-reflect+1)/2}">
+          <limit effort="${ThumbPitch3TorqueLimit}" lower="${ThumbPitch3PositionLimit_Lower}" upper="${ThumbPitch3PositionLimit_Upper}" velocity="${ThumbPitch3VelocityLimit}"/>
+        </xacro:if>
     </xacro:revolute_joint>
   </xacro:macro>
@@ -124,10 +139,10 @@
                           origin_rpy="${ThumbPitch3FrameOrientation_Roll} ${ThumbPitch3FrameOrientation_Pitch} ${ThumbPitch3FrameOrientation_Yaw}"/>
   </xacro:macro>
-  <xacro:macro name="v1_right_thumb_actuators" params="prefix api">
+  <xacro:macro name="right_thumb_actuators" params="prefix api">
     <xacro:v1_actuator name="${RTA1_Actuator_Name}" api="${api}" />
     <xacro:v1_actuator name="${RTA2_Actuator_Name}" api="${api}" />
     <xacro:v1_actuator name="${RTA3_Actuator_Name}" api="${api}" />
   </xacro:macro>
-  <xacro:macro name="v1_left_thumb_actuators" params="prefix api">
+  <xacro:macro name="left_thumb_actuators" params="prefix api">
     <xacro:v1_actuator name="${LTA1_Actuator_Name}" api="${api}" />
     <xacro:v1_actuator name="${LTA2_Actuator_Name}" api="${api}" />

File: resources/models/val_description/robots/valkyrie_A/xacro/waist/waist.xacro (robot description, xacro)
@@ -76,5 +76,5 @@
   </xacro:macro>
   <!-- Actuators -->
-  <xacro:macro name="v1_waist_actuators"  params="name1 type1 name2 type2 name3 type3">
+  <xacro:macro name="waist_actuators"  params="name1 type1 name2 type2 name3 type3">
     <actuator name="${name1}" type="${type1}"/>
     <actuator name="${name2}" type="${type2}"/>
