Commit message: ROSI-9: pulling in new changes from urdf, includes mass and inertia updates from Jordan. wont fixBamboo. pair: Jordan. had to change inertia for hokuyo link

File: resources/models/val_description/robots/common/generic_models.xacro (robot description, xacro)
@@ -43,8 +43,6 @@
         <geometry>
           <mesh filename="${visual_mesh}"/>
-          <!-- <cylinder radius="${radius}" length="${length}"/> -->
-        </geometry>
-        <origin rpy="0 0 0" xyz="0 0 0"/>
-        <!-- <origin rpy="${origin_rpy}" xyz="${origin_xyz}"/> -->
+        </geometry>
+        <origin rpy="0 0 0" xyz="0 0 0"/>
         <material name="${material}"/>
       </visual>
@@ -261,7 +259,4 @@
       </collision>
     </link>
-<!--    <gazebo reference="${name}">
-      <material>Gazebo/${material}</material>
-    </gazebo> -->
   </xacro:macro>
   <xacro:macro name="virtual_link_sphere" params="name radius mass origin_xyz origin_rpy">
@@ -297,8 +292,4 @@
     </link>
   </xacro:macro>
-  <!-- May 2015: However zero mass/inertials links are still useful. (And removed with gz sdf)
-  This macro here was added to allow fixed links to have (almost) no effect on the output compound
-  sdf mass and inertia
-  -->
   <xacro:property name="massless_virtual_link_mass" value="0.0000001"/>
   <xacro:property name="massless_virtual_link_radius" value="0.0000001"/>

File: resources/models/val_description/robots/valkyrie_A/xacro/arm/arm.xacro (robot description, xacro)
@@ -7,19 +7,16 @@
   <xacro:include filename="$(find val_description)/robots/valkyrie_A/xacro/arm/frame_parameters.xacro"/>
   <xacro:include filename="$(find val_description)/robots/valkyrie_A/xacro/arm/mass_parameters.xacro"/>
-  <xacro:property name="AJ1_Link_Width" value="0.202"/>
-  <xacro:property name="AJ1_Link_Height" value="0.162"/>
+  <xacro:property name="AJ1_Link_Width" value="0.162"/>
+  <xacro:property name="AJ1_Link_Height" value="0.202"/>
   <xacro:property name="AJ1_Link_Length" value="0.146"/>
-  <xacro:property name="AJ2_Link_Width" value="0.22179303376297454520"/>
-  <xacro:property name="AJ2_Link_Height" value="0.16373203016010165478"/>
-  <xacro:property name="AJ2_Link_Length" value="0.15560348965569942292"/>
-  <xacro:property name="AJ3_Link_Width" value="0.158"/>
-  <xacro:property name="AJ3_Link_Height" value="0.285"/>
-  <xacro:property name="AJ3_Link_Length" value="0.136"/>
+  <xacro:property name="AJ3_Link_Width" value="0.136"/>
+  <xacro:property name="AJ3_Link_Height" value="0.158"/>
+  <xacro:property name="AJ3_Link_Length" value="0.285"/>
   <xacro:property name="AJ4_Link_Width" value="0.11323257841518076516"/>
   <xacro:property name="AJ4_Link_Height" value="0.11855222975004402197"/>
   <xacro:property name="AJ4_Link_Length" value="0.10487312631734664603"/>
   <xacro:property name="AJ5_Link_Width" value="0.13557189311158912570"/>
-  <xacro:property name="AJ5_Link_Height" value="0.25365181285234167374"/>
-  <xacro:property name="AJ5_Link_Length" value="0.11439484172804967321"/>
+  <xacro:property name="AJ5_Link_Height" value="0.11439484172804967321"/>
+  <xacro:property name="AJ5_Link_Length" value="0.25365181285234167374"/>
   <xacro:property name="AJ6_Link_Width" value="0.03"/>
   <xacro:property name="AJ6_Link_Height" value="0.01"/>
@@ -29,5 +26,4 @@
   <xacro:property name="AJ7_Link_Length" value="0.038"/>
   <xacro:macro name="make_upper_arm" params="prefix reflect upper_arm_root_link">
-    <!-- LINKS -->
     <xacro:box_link name="${ShoulderPitchLinkName}"
                     width="${AJ1_Link_Width}" height="${AJ1_Link_Height}" depth="${AJ1_Link_Length}" mass="${ShoulderPitchLinkMass}"
@@ -36,7 +32,10 @@
                     material="Gold"
                     collision_mesh="${mesh_root}/arms/aj1_${prefix}.dae" />
-    <xacro:box_link name="${ShoulderRollLinkName}"
-                    width="${AJ2_Link_Width}" height="${AJ2_Link_Height}" depth="${AJ2_Link_Length}" mass="${ShoulderRollLinkMass}"
-                    origin_xyz="${ShoulderRollLinkComPosition}" origin_rpy="0 0 0"
+    <xacro:standard_link name="${ShoulderRollLinkName}"
+                    mass="${ShoulderRollLinkMass}"
+                    origin_xyz="${ShoulderRollLinkComPosition}"
+                    ixx="${ShoulderRollLinkInertia_IXX}" ixy="${ShoulderRollLinkInertia_IXY}" ixz="${ShoulderRollLinkInertia_IXZ}"
+                    iyy="${ShoulderRollLinkInertia_IYY}" iyz="${ShoulderRollLinkInertia_IYZ}" izz="${ShoulderRollLinkInertia_IZZ}"
+                    origin_rpy="0 0 0"
                     visual_mesh="${mesh_root}/arms/aj2_${prefix}.dae"
                     material="White"
@@ -55,5 +54,4 @@
                     material="Gold"
                     collision_mesh="${mesh_root}/arms/aj4_${prefix}.dae" />
-    <!-- AJ1 -->
     <xacro:revolute_joint_ex jointName="${ShoulderPitchJointName}"
                           parent="${upper_arm_root_link}" child="${ShoulderPitchLinkName}"
@@ -65,5 +63,4 @@
         <controller_gains Kp="20000" Kd="400"/>
     </xacro:revolute_joint_ex>
-    <!-- AJ2 -->
     <xacro:revolute_joint_ex jointName="${ShoulderRollJointName}"
                           parent="${ShoulderPitchLinkName}" child="${ShoulderRollLinkName}"
@@ -80,5 +77,4 @@
         <controller_gains Kp="20000" Kd="400"/>
     </xacro:revolute_joint_ex>
-    <!-- AJ3 -->
     <xacro:revolute_joint_ex jointName="${ShoulderYawJointName}"
                           parent="${ShoulderRollLinkName}" child="${ShoulderYawLinkName}"
@@ -90,5 +86,4 @@
         <controller_gains Kp="20000" Kd="400"/>
     </xacro:revolute_joint_ex>
-    <!-- AJ4 -->
     <xacro:revolute_joint_ex jointName="${ElbowPitchJointName}"
                           parent="${ShoulderYawLinkName}" child="${ElbowPitchLinkName}"
@@ -107,5 +102,4 @@
   </xacro:macro>
   <xacro:macro name="make_lower_arm" params="prefix reflect lower_arm_root_link">
-    <!-- LINKS -->
     <xacro:box_link name="${ForearmLinkName}"
                     width="${AJ5_Link_Width}" height="${AJ5_Link_Height}" depth="${AJ5_Link_Length}" mass="${ForearmYawLinkMass}"
@@ -129,5 +123,4 @@
                     material="Gold"
                     collision_mesh="${mesh_root}/arms/palm_${prefix}.dae"/>
-    <!-- AJ5 -->
     <xacro:revolute_joint_ex jointName="${ForearmYawJointName}"
                           parent="${lower_arm_root_link}" child="${ForearmLinkName}"
@@ -139,5 +132,4 @@
         <controller_gains Kp="20000" Kd="0"/>
     </xacro:revolute_joint_ex>
-    <!-- AJ6 -->
     <xacro:revolute_joint_ex jointName="${WristRollJointName}"
                           parent="${ForearmLinkName}" child="${WristRollLinkName}"
@@ -154,5 +146,4 @@
         <controller_gains Kp="20000" Kd="400"/>
     </xacro:revolute_joint_ex>
-    <!-- AJ7 -->
     <xacro:revolute_joint_ex jointName="${WristPitchJointName}"
                           parent="${WristRollLinkName}" child="${WristPitchLinkName}"
@@ -174,5 +165,4 @@
     <xacro:make_lower_arm prefix="${prefix}" reflect="${reflect}" lower_arm_root_link="${ElbowPitchLinkName}" />
   </xacro:macro>
-  <!-- Actuators -->
   <xacro:macro name="upper_arm_actuators" params="name1 type1 name2 type2 name3 type3 name4 type4">
     <actuator name="${name1}" type="${type1}"/>

File: resources/models/val_description/robots/valkyrie_A/xacro/arm/mass_parameters.xacro (robot description, xacro)
@@ -3,13 +3,25 @@
   <xacro:property name="ShoulderPitchLinkMass" value="2.65" />
   <xacro:property name="ShoulderPitchLinkComPosition" value="-0.012000 ${reflect*0.251000} 0.000000" />
-  <xacro:property name="ShoulderRollLinkMass" value="2.87" />
-  <xacro:property name="ShoulderRollLinkComPosition" value="-0.020086 ${reflect*0.040000} -0.004999" />
-  <xacro:property name="ShoulderYawLinkMass" value="2.575" />
-  <xacro:property name="ShoulderYawLinkComPosition" value="0.004000	${reflect*0.273000}	-0.019953" />
-  <xacro:property name="ElbowPitchLinkMass" value="2.367" />
-  <xacro:property name="ElbowPitchLinkComPosition" value="-0.027000	${reflect*0.080200} 0.000000" />
-  <xacro:property name="ForearmYawLinkMass" value="2.903" />
+  <xacro:property name="ShoulderRollLinkMass" value="3.970000" />
+  <xacro:property name="ShoulderRollLinkComPosition" value="-0.008513 ${reflect*0.020680} 0.001088" />
+  <xacro:property name="ShoulderRollLinkInertia_IXX" value="0.009494119" />
+  <xacro:property name="ShoulderRollLinkInertia_IXY" value="${reflect*0.000067294}" />
+  <xacro:property name="ShoulderRollLinkInertia_IXZ" value="${reflect*-0.000037177}" />
+  <xacro:property name="ShoulderRollLinkInertia_IYY" value="0.007680534" />
+  <xacro:property name="ShoulderRollLinkInertia_IYZ" value="0.000008874" />
+  <xacro:property name="ShoulderRollLinkInertia_IZZ" value="0.011454772" />
+  <xacro:property name="ShoulderYawLinkMass" value="3.085000" />
+  <xacro:property name="ShoulderYawLinkComPosition" value="-0.004304	${reflect*0.209832}	-0.007295" />
+  <xacro:property name="ShoulderYawLinkInertia_IXX" value="0.036063329" />
+  <xacro:property name="ShoulderYawLinkInertia_IXY" value="0.007025754" />
+  <xacro:property name="ShoulderYawLinkInertia_IXZ" value="${reflect*-0.000670432}" />
+  <xacro:property name="ShoulderYawLinkInertia_IYY" value="0.004652334" />
+  <xacro:property name="ShoulderYawLinkInertia_IYZ" value="${reflect*0.002512451}" />
+  <xacro:property name="ShoulderYawLinkInertia_IZZ" value="0.038329341" />
+  <xacro:property name="ElbowPitchLinkMass" value="1.830000" />
+  <xacro:property name="ElbowPitchLinkComPosition" value="-0.020344	${reflect*0.014722} -0.022300" />
+  <xacro:property name="ForearmYawLinkMass" value="2.476" />
   <xacro:property name="ForearmYawLinkComPosition" value="0.015000	${reflect*0.110000} 0.019564" />
-  <xacro:property name="WristRollLinkMass" value="0.1" />
+  <xacro:property name="WristRollLinkMass" value="0.14" />
   <xacro:property name="WristRollLinkComPosition" value="0 ${reflect*0} 0" />
   <xacro:property name="PalmMass" value="0.712" />

File: resources/models/val_description/robots/valkyrie_A/xacro/head/head.xacro (robot description, xacro)
@@ -18,7 +18,10 @@
                                     origin_rpy="0 0 0"
                                     mesh_filename="${mesh_root}/head/neckj2.dae"/>
-    <xacro:sphere_link name="${UpperNeckPitchLinkName}"
-                       radius="${NJ3_Link_Radius}" mass="${UpperNeckPitchLinkMass}"
-                       origin_xyz="${UpperNeckPitchLinkComPosition}" origin_rpy="0 0 0"
+    <xacro:standard_link name="${UpperNeckPitchLinkName}"
+                       mass="${UpperNeckPitchLinkMass}"
+                       origin_xyz="${UpperNeckPitchLinkComPosition}"
+                       ixx="${UpperNeckPitchLinkInertia_IXX}" ixy="${UpperNeckPitchLinkInertia_IXY}" ixz="${UpperNeckPitchLinkInertia_IXZ}"
+                       iyy="${UpperNeckPitchLinkInertia_IYY}" iyz="${UpperNeckPitchLinkInertia_IYZ}" izz="${UpperNeckPitchLinkInertia_IZZ}"
+                       origin_rpy="0 0 0"
                        visual_mesh="${mesh_root}/head/head_multisense_no_visor.dae"
                        material="White"
@@ -51,7 +54,11 @@
       <controller_gains Kp="20000" Kd="0"/>
     </xacro:revolute_joint_ex>
+  </xacro:macro>
+    <xacro:macro name="include_multisense_sim">
+      <xacro:fixed_joint jointName="multisense_head_root_joint" parent="${UpperNeckPitchLinkName}" child="head" origin_xyz="0.183585961 0.0 0.075353826" origin_rpy="-3.14159 0.130899694 0.0" />
     </xacro:macro>
-    <xacro:macro name="include_multisense">
-      <xacro:fixed_joint jointName="multisense_head_root" parent="${UpperNeckPitchLinkName}" child="head" origin_xyz="0.183585961 0.0 0.075353826" origin_rpy="-3.14159 0.130899694 0.0" />
+    <xacro:macro name="include_multisense_hw">
+      <xacro:massless_virtual_link name="multisense_root_link" origin_xyz="0 0 0" origin_rpy="0 0 0"/>
+      <xacro:fixed_joint jointName="multisense_head_root_joint" parent="${UpperNeckPitchLinkName}" child="multisense_root_link" origin_xyz="0.183585961 0.0 0.075353826" origin_rpy="-3.14159 0.130899694 0.0" />
     </xacro:macro>
   <xacro:macro name="neck_actuators" params="name1 type1 name2 type2 name3 type3">

File: resources/models/val_description/robots/valkyrie_A/xacro/head/joint_limits.xacro (robot description, xacro)
@@ -5,9 +5,9 @@
   <xacro:property name="UpperNeckPitchTorqueLimit" value="26" />
   <xacro:property name="LowerNeckPitchPositionLimit_Lower" value="0" />
-  <xacro:property name="NeckYawPositionLimit_Lower" value="-1.57" />
-  <xacro:property name="UpperNeckPitchPositionLimit_Lower" value="-0.087" />
+  <xacro:property name="NeckYawPositionLimit_Lower" value="-1.04719755" />
+  <xacro:property name="UpperNeckPitchPositionLimit_Lower" value="-0.872" />
   <xacro:property name="LowerNeckPitchPositionLimit_Upper" value="1.162" />
-  <xacro:property name="NeckYawPositionLimit_Upper" value="1.57" />
-  <xacro:property name="UpperNeckPitchPositionLimit_Upper" value="0.785" />
+  <xacro:property name="NeckYawPositionLimit_Upper" value="1.04719755" />
+  <xacro:property name="UpperNeckPitchPositionLimit_Upper" value="0.0" />
   <xacro:property name="LowerNeckPitchVelocityLimit" value="5" />
   <xacro:property name="NeckYawVelocityLimit" value="5" />

File: resources/models/val_description/robots/valkyrie_A/xacro/head/mass_parameters.xacro (robot description, xacro)
@@ -1,10 +1,16 @@
 <?xml version="1.0" ?>
 <robot xmlns:xacro="http://www.ros.org/wiki/xacro" name="v1/head/mass_parameters">
-  <xacro:property name="LowerNeckPitchLinkMass" value="0.471" />
+  <xacro:property name="LowerNeckPitchLinkMass" value="1.05" />
   <xacro:property name="LowerNeckPitchLinkComPosition" value="0 0 0" />
   <xacro:property name="NeckYawLinkMass" value="1.4" />
   <xacro:property name="NeckYawLinkComPosition" value="0 0 0" />
-  <xacro:property name="UpperNeckPitchLinkMass" value="4.06" />
+  <xacro:property name="UpperNeckPitchLinkMass" value="4.59" />
   <xacro:property name="UpperNeckPitchLinkComPosition" value="0.091874 0.001012 -0.005277" />
+  <xacro:property name="UpperNeckPitchLinkInertia_IXX" value="0.041442523" />
+  <xacro:property name="UpperNeckPitchLinkInertia_IXY" value="-0.000055137" />
+  <xacro:property name="UpperNeckPitchLinkInertia_IXZ" value="0.000287605" />
+  <xacro:property name="UpperNeckPitchLinkInertia_IYY" value="0.044208496" />
+  <xacro:property name="UpperNeckPitchLinkInertia_IYZ" value="0.000245121" />
+  <xacro:property name="UpperNeckPitchLinkInertia_IZZ" value="0.041961853" />
   <xacro:property name="HokuyoLinkMass" value="0.057664"/>
   <xacro:property name="HokuyoLinkComPosition" value="0.14793 0.0 0.01"/>

File: resources/models/val_description/robots/valkyrie_A/xacro/leg/leg.xacro (robot description, xacro)
@@ -14,19 +14,4 @@
   <xacro:property name="LJ1_Link_Origin_Y" value="0.0013"/>
   <xacro:property name="LJ1_Link_Origin_Z" value="0.03867"/>
-  <xacro:property name="LJ2_Link_Width" value="0.123"/>
-  <xacro:property name="LJ2_Link_Height" value="0.131"/>
-  <xacro:property name="LJ2_Link_Length" value="0.185"/>
-  <xacro:property name="LJ3_Link_Width" value="0.24253719562602335524"/>
-  <xacro:property name="LJ3_Link_Height" value="0.18520578950459243295"/>
-  <xacro:property name="LJ3_Link_Length" value="0.55419965909040602714"/>
-  <xacro:property name="LJ4_Link_Box_Width" value="0.20288766696230062236"/>
-  <xacro:property name="LJ4_Link_Box_Height" value="0.20551228016178813007"/>
-  <xacro:property name="LJ4_Link_Box_Length" value="0.44528684954574881960"/>
-  <xacro:property name="LJ5_Link_Width" value="0.033"/>
-  <xacro:property name="LJ5_Link_Height" value="0.076"/>
-  <xacro:property name="LJ5_Link_Length" value="0.025"/>
-  <xacro:property name="LJ6_Link_Width" value="0.300"/>
-  <xacro:property name="LJ6_Link_Height" value="0.128"/>
-  <xacro:property name="LJ6_Link_Length" value="0.082"/>
   <xacro:macro name="make_leg_links" params="prefix reflect leg_root_link">
     <xacro:box_link name="${HipYawLinkName}"
@@ -36,35 +21,45 @@
                     material="Gold"
                     collision_mesh="${mesh_root}/legs/lj1_${prefix}.dae"/>
-    <xacro:box_link name="${HipRollLinkName}"
-                    width="${LJ2_Link_Width}" height="${LJ2_Link_Height}" depth="${LJ2_Link_Length}" mass="${HipRollLinkMass}"
+    <xacro:standard_link name="${HipRollLinkName}"
+                    mass="${HipRollLinkMass}"
                     origin_xyz="${HipRollLinkComPosition}"
+                    ixx="${HipRollLinkInertia_IXX}" ixy="${HipRollLinkInertia_IXY}" ixz="${HipRollLinkInertia_IXZ}"
+                    iyy="${HipRollLinkInertia_IYY}" iyz="${HipRollLinkInertia_IYZ}" izz="${HipRollLinkInertia_IZZ}"
                     origin_rpy="0 0 0"
                     visual_mesh="${mesh_root}/legs/lj2_${prefix}.dae"
                     material="White"
                     collision_mesh="${mesh_root}/legs/lj2_${prefix}.dae"/>
-    <xacro:box_link name="${HipPitchLinkName}"
-                    width="${LJ3_Link_Width}" height="${LJ3_Link_Height}" depth="${LJ3_Link_Length}" mass="${HipPitchLinkMass}"
+    <xacro:standard_link name="${HipPitchLinkName}"
+                    mass="${HipPitchLinkMass}"
                     origin_xyz="${HipPitchLinkComPosition}"
+                    ixx="${HipPitchLinkInertia_IXX}" ixy="${HipPitchLinkInertia_IXY}" ixz="${HipPitchLinkInertia_IXZ}"
+                    iyy="${HipPitchLinkInertia_IYY}" iyz="${HipPitchLinkInertia_IYZ}" izz="${HipPitchLinkInertia_IZZ}"
                     origin_rpy="0 0 0"
                     visual_mesh="${mesh_root}/legs/lj3_${prefix}.dae"
                     material="White"
                     collision_mesh="${mesh_root}/legs/lj3_${prefix}.dae"/>
-    <xacro:box_link name="${KneePitchLinkName}"
-                    width="${LJ4_Link_Box_Width}" height="${LJ4_Link_Box_Height}" depth="${LJ4_Link_Box_Length}" mass="${KneePitchLinkMass}"
+    <xacro:standard_link name="${KneePitchLinkName}"
+                    mass="${KneePitchLinkMass}"
                     origin_xyz="${KneePitchLinkComPosition}"
+                    ixx="${KneePitchLinkInertia_IXX}" ixy="${KneePitchLinkInertia_IXY}" ixz="${KneePitchLinkInertia_IXZ}"
+                    iyy="${KneePitchLinkInertia_IYY}" iyz="${KneePitchLinkInertia_IYZ}" izz="${KneePitchLinkInertia_IZZ}"
                     origin_rpy="0 0 0"
                     visual_mesh="${mesh_root}/legs/lj4_${prefix}.dae"
                     material="White"
                     collision_mesh="${mesh_root}/legs/lj4_${prefix}.dae"/>
-    <xacro:box_link name="${AnklePitchLinkName}"
-                    width="${LJ5_Link_Width}" height="${LJ5_Link_Height}" depth="${LJ5_Link_Length}" mass="${AnklePitchLinkMass}"
+    <xacro:standard_link name="${AnklePitchLinkName}"
+                    mass="${AnklePitchLinkMass}"
                     origin_xyz="${AnklePitchLinkComPosition}"
+                    ixx="${AnklePitchLinkInertia_IXX}" ixy="${AnklePitchLinkInertia_IXY}" ixz="${AnklePitchLinkInertia_IXZ}"
+                    iyy="${AnklePitchLinkInertia_IYY}" iyz="${AnklePitchLinkInertia_IYZ}" izz="${AnklePitchLinkInertia_IZZ}"
                     origin_rpy="0 0 0"
                     visual_mesh="${mesh_root}/legs/lj5.dae"
                     material="White"
                     collision_mesh="${mesh_root}/legs/lj5.dae"/>
-    <xacro:box_link name="${AnkleRollLinkName}"
-                    width="${LJ6_Link_Width}" height="${LJ6_Link_Height}" depth="${LJ6_Link_Length}" mass="${FootMass}"
+    <xacro:standard_link name="${AnkleRollLinkName}"
+                    mass="${FootMass}"
                     origin_xyz="${FootComPosition}"
+                    ixx="${FootInertia_IXX}" ixy="${FootInertia_IXY}" ixz="${FootInertia_IXZ}"
+                    iyy="${FootInertia_IYY}" iyz="${FootInertia_IYZ}" izz="${FootInertia_IZZ}"
                     origin_rpy="0 0 0"
                     visual_mesh="${mesh_root}/legs/foot_${prefix}.dae"
@@ -73,5 +68,4 @@
   </xacro:macro>
   <xacro:macro name="make_leg_joints" params="prefix reflect leg_root_link">
-    <!-- LJ1 -->
     <xacro:revolute_joint_ex jointName="${HipYawJointName}"
                           parent="${HipYawParentLinkName}" child="${HipYawLinkName}"
@@ -146,5 +140,4 @@
     <xacro:make_ankle_joints prefix="${prefix}" reflect="${reflect}" leg_root_link="${leg_root_link}" />
   </xacro:macro>
-  <!-- Sensors -->
   <xacro:macro name="v1_leg_sensors" params="prefix reflect">
     <xacro:virtual_fixed_frame_offset name="${prefix}COP"
