Commit message: ROSI-9: pulling in new changes from urdf, includes mass and inertia updates from Jordan. wont fixBamboo. pair: Jordan. had to change inertia for hokuyo link

File: resources/models/val_description/robots/valkyrie_A/xacro/leg/mass_parameters.xacro (robot description, xacro)
@@ -1,15 +1,45 @@
 <?xml version="1.0" ?>
-<robot xmlns:xacro="http://www.ros.org/wiki/xacro" name="v1/leg/mass_parameters">
+<robot xmlns:xacro="http://www.ros.org/wiki/xacro" name="leg_mass_parameters">
   <xacro:property name="HipYawLinkMass" value="2.39" />
   <xacro:property name="HipYawLinkComPosition" value="0.02176 ${reflect*-0.00131} 0.03867" />
-  <xacro:property name="HipRollLinkMass" value="5.95" />
-  <xacro:property name="HipRollLinkComPosition" value="-0.00185 ${reflect*0.02426} -0.019260" />
-  <xacro:property name="HipPitchLinkMass" value="10.3" />
-  <xacro:property name="HipPitchLinkComPosition" value="0.000057 ${reflect*0.050000} -0.220000" />
-  <xacro:property name="KneePitchLinkMass" value="7.4" />
-  <xacro:property name="KneePitchLinkComPosition" value="-0.004670 ${reflect*0.0050000} -0.184940" />
-  <xacro:property name="AnklePitchLinkMass" value="0.395" />
-  <xacro:property name="AnklePitchLinkComPosition" value="-0.001270 ${reflect*0.000000} -0.006010" />
-  <xacro:property name="FootMass" value="1.888" />
-  <xacro:property name="FootComPosition" value="0.068860 ${reflect*-0.000285} -0.051830" />
+  <xacro:property name="HipRollLinkMass" value="3.665000" />
+  <xacro:property name="HipRollLinkComPosition" value="0.012959 ${reflect*0.007550} -0.015950" />
+  <xacro:property name="HipRollLinkInertia_IXX" value="0.005978962" />
+  <xacro:property name="HipRollLinkInertia_IXY" value="${reflect*-0.000234823}" />
+  <xacro:property name="HipRollLinkInertia_IXZ" value="0.000553962" />
+  <xacro:property name="HipRollLinkInertia_IYY" value="0.009372646" />
+  <xacro:property name="HipRollLinkInertia_IYZ" value="${reflect*0.000778956}" />
+  <xacro:property name="HipRollLinkInertia_IZZ" value="0.008193117" />
+  <xacro:property name="HipPitchLinkMass" value="10.20" />
+  <xacro:property name="HipPitchLinkComPosition" value="0.016691 ${reflect*0.091397} -0.207875" />
+  <xacro:property name="HipPitchLinkInertia_IXX" value="0.240834130" />
+  <xacro:property name="HipPitchLinkInertia_IXY" value="${reflect*0.000035915}" />
+  <xacro:property name="HipPitchLinkInertia_IXZ" value="0.003699383" />
+  <xacro:property name="HipPitchLinkInertia_IYY" value="0.256897050" />
+  <xacro:property name="HipPitchLinkInertia_IYZ" value="${reflect*-0.001333005}" />
+  <xacro:property name="HipPitchLinkInertia_IZZ" value="0.023276352" />
+  <xacro:property name="KneePitchLinkMass" value="6.600000" />
+  <xacro:property name="KneePitchLinkComPosition" value="0.002425 -0.001543 -0.189511" />
+  <xacro:property name="KneePitchLinkInertia_IXX" value="0.096117529" />
+  <xacro:property name="KneePitchLinkInertia_IXY" value="0.000107885" />
+  <xacro:property name="KneePitchLinkInertia_IXZ" value="0.006319047" />
+  <xacro:property name="KneePitchLinkInertia_IYY" value="0.097118447" />
+  <xacro:property name="KneePitchLinkInertia_IYZ" value="-0.000494739" />
+  <xacro:property name="KneePitchLinkInertia_IZZ" value="0.013722874" />
+  <xacro:property name="AnklePitchLinkMass" value="0.06" />
+  <xacro:property name="AnklePitchLinkComPosition" value="-0.001269 0.00009 -0.006013" />
+  <xacro:property name="AnklePitchLinkInertia_IXX" value="0.000011226" />
+  <xacro:property name="AnklePitchLinkInertia_IXY" value="0.000000000" />
+  <xacro:property name="AnklePitchLinkInertia_IXZ" value="0.000002735" />
+  <xacro:property name="AnklePitchLinkInertia_IYY" value="0.000026700" />
+  <xacro:property name="AnklePitchLinkInertia_IYZ" value="0.0" />
+  <xacro:property name="AnklePitchLinkInertia_IZZ" value="0.000018792" />
+  <xacro:property name="FootMass" value="3.2550" />
+  <xacro:property name="FootComPosition" value="0.040004 -0.00381 -0.049558" />
+  <xacro:property name="FootInertia_IXX" value="0.008966273" />
+  <xacro:property name="FootInertia_IXY" value="-0.000086029" />
+  <xacro:property name="FootInertia_IXZ" value="0.003944774" />
+  <xacro:property name="FootInertia_IYY" value="0.023943858" />
+  <xacro:property name="FootInertia_IYZ" value="0.000105218" />
+  <xacro:property name="FootInertia_IZZ" value="0.028128777" />
 </robot>

File: resources/models/val_description/robots/valkyrie_A/xacro/pelvis/pelvis.xacro (robot description, xacro)
@@ -2,7 +2,9 @@
     <xacro:property name="Pelvis_Link_Name" value="Pelvis" />
     <xacro:macro name="make_pelvis">
-        <xacro:box_link name="${Pelvis_Link_Name}"
-                        width="0.28251052337959348115" height="0.34445341259705453130" depth="0.36811588436650161116" mass="6.986"
-                        origin_xyz="0.000733954 -0.000895362 -0.0702552"
+        <xacro:standard_link name="${Pelvis_Link_Name}"
+                        mass="8.22"
+                        origin_xyz="-0.00532 -0.003512 -0.0036"
+                        ixx="0.11866378" ixy="-0.000143482" ixz="0.003271293"
+                        iyy="0.097963425" iyz="0.002159545" izz="0.083854638"
                         origin_rpy="0 0 0"
                         visual_mesh="${mesh_root}/pelvis/pelvis.dae" material="White"

File: resources/models/val_description/robots/valkyrie_A/xacro/waist/mass_parameters.xacro (robot description, xacro)
@@ -2,5 +2,14 @@
 <robot xmlns:xacro="http://www.ros.org/wiki/xacro" name="v1/waist/mass_parameters">
 	<xacro:property name="TorsoYawLinkMass" value="2.858" />
+	<xacro:property name="TorsoYawLinkComPosition" value="0.0 0.0 0.0" />
 	<xacro:property name="TorsoPitchLinkMass" value="0.001"/>
-  <xacro:property name="TorsoRollLinkMass" value="42.6" />
+	<xacro:property name="TorsoPitchLinkComPosition" value="0.0 0.0 0.0" />
+  <xacro:property name="TorsoRollLinkMass" value="39.470000" />
+  <xacro:property name="TorsoRollLinkComPosition" value="-0.178048 0.012293 0.238350" />
+  <xacro:property name="TorsoRollLinkInertia_IXX" value="0.874514000" />
+  <xacro:property name="TorsoRollLinkInertia_IXY" value="0.039067696" />
+  <xacro:property name="TorsoRollLinkInertia_IXZ" value="0.088824164" />
+  <xacro:property name="TorsoRollLinkInertia_IYY" value="1.271005200" />
+  <xacro:property name="TorsoRollLinkInertia_IYZ" value="-0.004025467" />
+  <xacro:property name="TorsoRollLinkInertia_IZZ" value="1.056875300" />
 </robot>

File: resources/models/val_description/robots/valkyrie_A/xacro/waist/waist.xacro (robot description, xacro)
@@ -1,3 +1,3 @@
-<robot xmlns:xacro="http://www.ros.org/wiki/xacro" name="waist">
+<robot xmlns:xacro="http://www.ros.org/wiki/xacro" name="v1/waist">
   <!-- Properties -->
   <xacro:include filename="$(find val_description)/robots/valkyrie_A/xacro/waist/joint_names.xacro"/>
@@ -10,7 +10,4 @@
   <xacro:include filename="$(find val_description)/robots/common/sensors/microstrain.xacro"/>
   <xacro:include filename="$(find val_description)/robots/common/sensors/flea.xacro"/>
-  <xacro:property name="Trunk_Width" value="0.42203731228144558685"/>
-  <xacro:property name="Trunk_Height" value="0.39817895332782154982"/>
-  <xacro:property name="Trunk_Length" value="0.47605775481079287692"/>
   <xacro:macro name="make_waist_common" params="waist_root_link">
     <xacro:revolute_joint_ex jointName="${TorsoYawJointName}"
@@ -57,8 +54,10 @@
                     material="White"
                     collision_mesh="${mesh_root}/torso/torsopitch.dae" />
-    <xacro:box_link name="${TorsoRollLinkName}"
-                    width="${Trunk_Width}" height="${Trunk_Height}" depth="${Trunk_Length}" mass="${TorsoRollLinkMass}"
+    <xacro:standard_link name="${TorsoRollLinkName}"
+                    mass="${TorsoRollLinkMass}"
+                    ixx="${TorsoRollLinkInertia_IXX}" ixy="${TorsoRollLinkInertia_IXY}" ixz="${TorsoRollLinkInertia_IXZ}"
+                    iyy="${TorsoRollLinkInertia_IYY}" iyz="${TorsoRollLinkInertia_IYZ}" izz="${TorsoRollLinkInertia_IZZ}"
                     origin_rpy="0 0 0"
-                    origin_xyz="-0.0981 0.0 0.255"
+                    origin_xyz="${TorsoRollLinkComPosition}"
                     visual_mesh="${mesh_root}/torso/torso.dae"
                     material="White"
@@ -75,5 +74,4 @@
                     collision_mesh="${mesh_root}/torso/wj3.dae" />
   </xacro:macro>
-  <!-- Actuators -->
   <xacro:macro name="waist_actuators"  params="name1 type1 name2 type2 name3 type3">
     <actuator name="${name1}" type="${type1}"/>

File: resources/models/val_description/urdf/valkyrie_A_hw.urdf (robot description, URDF)
Before this commit: robot valkyrie, 69 links, 68 joints
Links:
- added link multisense_root_link, mass 1e-07
- link LeftAnklePitchLink: mass 0.395 -> 0.06
- link LeftElbowPitchLink: mass 2.367 -> 1.83
- link LeftFoot: mass 1.888 -> 3.255
- link LeftForearmLink: mass 2.903 -> 2.476
- link LeftHipPitchLink: mass 10.3 -> 10.2
- link LeftHipRollLink: mass 5.95 -> 3.665
- link LeftKneePitchLink: mass 7.4 -> 6.6
- link LeftShoulderRollLink: mass 2.87 -> 3.97
- link LeftShoulderYawLink: mass 2.575 -> 3.085
- link LeftWristRollLink: mass 0.1 -> 0.14
- link Pelvis: mass 6.986 -> 8.22
- link RightAnklePitchLink: mass 0.395 -> 0.06
- link RightElbowPitchLink: mass 2.367 -> 1.83
- link RightFoot: mass 1.888 -> 3.255
- link RightForearmLink: mass 2.903 -> 2.476
- link RightHipPitchLink: mass 10.3 -> 10.2
- link RightHipRollLink: mass 5.95 -> 3.665
- link RightKneePitchLink: mass 7.4 -> 6.6
- link RightShoulderRollLink: mass 2.87 -> 3.97
- link RightShoulderYawLink: mass 2.575 -> 3.085
- link RightWristRollLink: mass 0.1 -> 0.14
- link Torso: mass 42.6 -> 39.47
- link UpperNeckPitchLinkName: mass 4.06 -> 4.59
Joints:
- added joint multisense_head_root_joint: type fixed, parent UpperNeckPitchLinkName, child multisense_root_link, origin xyz=0.183585961 0.0 0.075353826 rpy=-3.14159 0.130899694 0.0, axis 0 0 1
- joint NeckYaw: limit lower=-1.57 upper=1.57 effort=26 velocity=5 -> lower=-1.04719755 upper=1.04719755 effort=26 velocity=5
- joint UpperNeckPitch: limit lower=-0.087 upper=0.785 effort=26 velocity=5 -> lower=-0.872 upper=0.0 effort=26 velocity=5
