Commit message: ROSI-27: generated urdfs and sdfs from latest xacros; won't fixbamboo

File: resources/models/val_description/robots/valkyrie_A/xacro/head/link_names.xacro (robot description, xacro)
@@ -4,4 +4,4 @@
   <xacro:property name="LowerNeckPitchLinkName" value="LowerNeckPitchLink" />
   <xacro:property name="NeckYawLinkName" value="NeckYawLink" />
-  <xacro:property name="UpperNeckPitchLinkName" value="UpperNeckPitchLinkName" />
+  <xacro:property name="UpperNeckPitchLinkName" value="UpperNeckPitchLink" />
 </robot>

File: resources/models/val_description/urdf/valkyrie_A_hw.urdf (robot description, URDF)
Before this commit: robot valkyrie, 70 links, 69 joints
Links:
- removed link UpperNeckPitchLinkName
- added link UpperNeckPitchLink, mass 4.59; collision mesh filename=package://val_description/meshes/head/head_multisense_no_vi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; visual mesh filename=package://val_description/meshes/head/head_multisense_no_vi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
Joints:
- joint UpperNeckPitch: child UpperNeckPitchLinkName -> UpperNeckPitchLink
- joint multisense_head_root_joint: parent UpperNeckPitchLinkName -> UpperNeckPitchLink
